File: mixer.kicad_sch (KiCad schematic)
At the start: 40 parts, among them T1 RF_BALUN, T2 RF_BALUN, U4 RFFC5072, U5 FM8625H, U6 FM8625H

Commit message: AC-couple RX analog baseband
Parts:
- R4: value 51k -> 51k±1%
Other:
- note removed: "1%"
Changed lines of the file:
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@@
-		)
-	)
-	(text "1%"
-		(exclude_from_sim no)
-		(at 162.56 99.06 0)
-		(effects
-			(font
-				(size 1.016 1.016)
-			)
-			(justify left bottom)
 		)
 	)
@@
 		(fields_autoplaced yes)
 		(property "Reference" "R4"
-			(at 162.56 104.14 90)
-			(effects
-				(font
-					(size 1.27 1.27)
-				)
-			)
-		)
-		(property "Value" "51k"
-			(at 162.56 106.68 90)
-			(effects
-				(font
+			(at 162.56 93.98 90)
+			(effects
+				(font
+					(size 1.27 1.27)
+				)
+			)
+		)
+		(property "Value" "51k±1%"
+			(at 162.56 96.52 90)
+			(effects
+				(font
