File: switch_control.kicad_sch (KiCad schematic)
At the start: 27 parts, among them U10 74LVC1G86, U11 74LVC1G86, U26 74HC00, U27 74LVC1G32

Commit message: Use mixer compensation amp only for TX
Parts:
- added C212: 1 uF, Capacitor_SMD:C_0201_0603Metric, symbol Device:C
- added TP66: TestPoint, TestPoint:TestPoint_Pad_D1.0mm, symbol Connector:TestPoint
- added U39: 74LVC1G08, Package_TO_SOT_SMD:SOT-353_SC-70-5, symbol 74xGxx:74LVC1G08
Connections:
- net GND: now also C212.2, U39.3 (GND)
- net MIX_EN: now also U39.1
- net TX_EN: now also U39.2
- new net TX_MIX_EN: TP66.1, U39.4
- new net VAA: C212.1, U39.5 (VCC)
Other:
- moved on the sheet: C24, C26, C27, C30, R24, R92, R94, R95, R96, R97, R98, R99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
