File: switch_control.kicad_sch (KiCad schematic)
At the start: 30 parts, among them U10 74LVC1G86, U11 74LVC1G86, U26 74HC00, U27 74LVC1G32, U39 74LVC1G08

Commit message: Drop 66 testpoint footprints from board; KiCad 10 format upgrade
Parts:
- removed TP35, TP37, TP38, TP39, TP40, TP41, TP42, TP43, TP44, TP45, TP46, TP66: TestPoint, TestPoint:TestPoint_Pad_D1.0mm, symbol Connector:TestPoint
Connections:
- net at R24.2, R92.1, U26.2: no longer U26.12

Commit message: Modules Merged. Power pours merged and edited. Inter-module routes to be completed.
Connections:
- net at U26.12: now also R24.2, R92.1, U26.2
Changed lines of the file:
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@@
 		(title "${TITLE}")
 		(date "${DATE}")
-		(rev "${VERSION}")
+		(rev "1")
 		(company "${COPYRIGHT}")
 		(comment 1 "${LICENSE}")
@@
 		)
 		(stroke
+			(width 0)
+			(type default)
+		)
+	)
+	(wire
+		(pts
+			(xy 71.12 151.13) (xy 106.68 151.13)
+		)
+		(stroke
