File: image_reject.kicad_sch (KiCad schematic)
At the start: 21 parts, among them U1 MXD8546F, U9 BGS13SN8

Commit message: Change SP3T RF switches from BGS13SN8 to MXD8638C
Parts:
- U9: value BGS13SN8 -> MXD8638C; footprint praline:TSNP-9-3 -> praline:MXD8638C; symbol praline:BGS13SN8 -> praline:MXD8638; Manufacturer Infineon -> Maxscend; Part Number BGS13SN8E6327XTSA1 -> MXD8638C
Connections:
- net 2V5RF: now also U9.7 (VDD); no longer U9.1 (VDD)
- net GND: now also U9.6 (GND); no longer U9.8 (GND)
- net LPF_OR_MIX_BYPASS: now also U9.8 (V2); no longer U9.2 (V2)
- net MIX_BYPASS: now also U9.5 (RF2); no longer U9.7 (RF2)
- net MIX_EN: now also U9.1 (V1); no longer U9.3 (V1)
- net RF: now also U9.4 (ANT); no longer U9.6 (RFin)
- net at C61.1, L15.1: now also U9.2 (RF3); no longer U9.4 (RF3)
- net at C96.2: now also U9.3 (RF1); no longer U9.5 (RF1)
Changed lines of the file:
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@@
 	)
 	(symbol
-		(lib_id "praline:BGS13SN8")
+		(lib_id "praline:MXD8638")
 		(at 219.71 64.77 0)
 		(unit 1)
@@
 			)
 		)
-		(property "Value" "BGS13SN8"
+		(property "Value" "MXD8638C"
 			(at 199.39 62.23 0)
 			(effects
@@
 			)
 		)
-		(property "Footprint" "praline:TSNP-9-3"
+		(property "Footprint" "praline:MXD8638C"
 			(at 219.71 64.77 0)
 			(effects
@@
 			)
 		)
-		(property "Datasheet" "https://www.infineon.com/dgdl/Infineon-BGS13SN8-DS-v02_02-EN.pdf?fileId=5546d462584d1d4a0158cf52e3ae03a7"
+		(property "Datasheet" "~"
 			(at 219.71 64.77 0)
 			(effects
@@
 			)
 		)
-		(property "Manufacturer" "Infineon"
+		(property "Manufacturer" "Maxscend"
 			(at 219.71 64.77 0)
 			(effects
@@
 			)
 		)
-		(property "Part Number" "BGS13SN8E6327XTSA1"
+		(property "Part Number" "MXD8638C"
 			(at 219.71 64.77 0)
 			(effects
