File: usb.kicad_sch (KiCad schematic)
At the start: 10 parts, among them J1 USB_C, U15 TVS_USB

Commit message: Merge phase 1: block schematics into parent; additive project metadata merge
Copied each block's edited sheet into the parent project (top-level
q-radio.kicad_sch untouched). Merged net classes (Power, diff85) with
their netclass patterns, unioned pre-defined track/via/diff-pair sizes,
and relaxed min_through_hole_diameter 0.3 -> 0.2032 to retain the
mcu/mixer via drills (flagged for fab confirmation). Adds
scripts/merge_blocks.py and the merge instructions document.

Co-Authored-By: Claude Fable 5 <noreply@anthropic.com>
Claude-Session: https://claude.ai/code/session_015o4bRsqK4wrTrSfjfByspi
Connections:
- net CC1: now also U15.2, U15.9 (NC); no longer U15.1, U15.10 (NC)
- net CC2: now also U15.1, U15.10 (NC); no longer U15.2, U15.9 (NC)
- net D+: now also FL1.2; no longer FL1.4
- net D-: now also FL1.4; no longer FL1.2
- net USB_DATA.D+: now also FL1.1; no longer FL1.3
- net USB_DATA.D-: now also FL1.3; no longer FL1.1
Other:
- moved on the sheet: FL1
Changed lines of the file:
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@@
 	)
 	(junction
-		(at 123.19 102.87)
+		(at 120.65 102.87)
+		(diameter 0)
+		(color 0 0 0 0)
+	)
+	(junction
+		(at 153.67 107.95)
+		(diameter 0)
+		(color 0 0 0 0)
+	)
+	(junction
+		(at 105.41 123.19)
 		(diameter 0)
 		(color 0 0 0 0)
@@
 	)
 	(junction
-		(at 128.27 97.79)
+		(at 156.21 123.19)
 		(diameter 0)
 		(color 0 0 0 0)
 	)
 	(junction
-		(at 105.41 123.19)
+		(at 105.41 85.09)
 		(diameter 0)
 		(color 0 0 0 0)
 	)
 	(junction
-		(at 120.65 97.79)
+		(at 105.41 120.65)
+		(diameter 0)
+		(color 0 0 0 0)
+	)
+	(junction
+		(at 156.21 97.79)
+		(diameter 0)
+		(color 0 0 0 0)
+	)
+	(junction
+		(at 123.19 97.79)
+		(diameter 0)
+		(color 0 0 0 0)
+	)
+	(junction
+		(at 149.86 55.88)
+		(diameter 0)
+		(color 0 0 0 0)
+	)
+	(junction
+		(at 172.72 55.88)
 		(diameter 0)
 		(color 0 0 0 0)
@@
 	)
 	(junction
-		(at 105.41 85.09)
-		(diameter 0)
-		(color 0 0 0 0)
-	)
-	(junction
-		(at 105.41 120.65)
-		(diameter 0)
-		(color 0 0 0 0)
-	)
-	(junction
-		(at 153.67 107.95)
-		(diameter 0)
-		(color 0 0 0 0)
-	)
-	(junction
-		(at 156.21 97.79)
-		(diameter 0)
-		(color 0 0 0 0)
-	)
-	(junction
-		(at 149.86 55.88)
-		(diameter 0)
-		(color 0 0 0 0)
-	)
-	(junction
-		(at 172.72 55.88)
-		(diameter 0)
-		(color 0 0 0 0)
-	)
-	(junction
-		(at 156.21 123.19)
+		(at 128.27 97.79)
 		(diameter 0)
 		(color 0 0 0 0)
@@
 	(wire
 		(pts
-			(xy 123.19 102.87) (xy 123.19 113.03)
+			(xy 123.19 97.79) (xy 128.27 97.79)
 		)
 		(stroke
@@
 	(wire
 		(pts
+			(xy 120.65 102.87) (xy 128.27 102.87)
+		)
+		(stroke
+			(width 0)
+			(type default)
+		)
+	)
+	(wire
+		(pts
 			(xy 128.27 102.87) (xy 128.27 107.95)
 		)
@@
 	(wire
 		(pts
+			(xy 123.19 97.79) (xy 123.19 113.03)
+		)
+		(stroke
+			(width 0)
+			(type default)
+		)
+	)
+	(wire
+		(pts
 			(xy 156.21 92.71) (xy 156.21 97.79)
 		)
@@
 	(wire
 		(pts
-			(xy 123.19 66.04) (xy 123.19 102.87)
+			(xy 123.19 66.04) (xy 123.19 97.79)
 		)
 		(stroke
@@
 	(wire
 		(pts
-			(xy 120.65 97.79) (xy 120.65 55.88)
-		)
-		(stroke
-			(width 0)
-			(type default)
-		)
-	)
-	(wire
-		(pts
-			(xy 120.65 97.79) (xy 120.65 110.49)
+			(xy 120.65 55.88) (xy 120.65 102.87)
 		)
 		(stroke
@@
 	(wire
 		(pts
-			(xy 120.65 97.79) (xy 128.27 97.79)
-		)
-		(stroke
-			(width 0)
-			(type default)
-		)
-	)
-	(wire
-		(pts
-			(xy 123.19 102.87) (xy 128.27 102.87)
+			(xy 120.65 102.87) (xy 120.65 110.49)
 		)
 		(stroke
@@
 	(symbol
 		(lib_id "Device:Filter_EMI_CommonMode")
-		(at 166.37 120.65 0)
-		(mirror y)
+		(at 166.37 120.65 180)
 		(unit 1)
 		(body_style 1)
@@
 		(dnp no)
 		(property "Reference" "FL1"
-			(at 166.37 115.57 0)
+			(at 165.608 114.808 0)
 			(show_name no)
 			(do_not_autoplace no)
@@
 		)
 		(property "Value" "CommonModeChoke"
-			(at 166.37 125.73 0)
+			(at 167.132 126.238 0)
 			(show_name no)
 			(do_not_autoplace no)
@@
 		)
 		(property "Footprint" "praline:L_CommonModeChoke_Murata_DLM0NS"
-			(at 166.37 119.634 0)
+			(at 166.37 121.666 0)
 			(hide yes)
 			(show_name no)
@@
 		)
 		(property "Datasheet" "https://www.murata.com/en-global/products/productdata/8799424610334/EFLD0009.pdf"
-			(at 166.37 119.634 0)
-			(hide yes)
-			(show_name no)
+			(at 166.37 121.666 0)
+			(hide yes)
+			(show_name no)
