File: LED_SW.kicad_sch (KiCad schematic)
At the start: 26 parts, among them SW1 SWITCH, SW2 SWITCH

Commit message: Modules Merged. Power pours merged and edited. Inter-module routes to be completed.
Other:
- title: (none) -> ${TITLE}
Changed lines of the file:
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@@
 	(paper "A4" portrait)
 	(title_block
+		(title "${TITLE}")
+		(rev "1")
 		(company "${COPYRIGHT}")
 		(comment 1 "${LICENSE}")
