File: clock/q-radio.kicad_pcb (KiCad board)
At the start: 6 copper layers, 68.6 x 34.3 mm, 40 parts, among them P1 SMA, P2 SMA, U19 SI5351C, U30 74LVC1G3157, U31 74LVC1G3157, U33 74HC4051, U37 74LVC1G3157, X1 TCXO

Commit message: All sub-modules added to child projects
Parts:
- removed FID1, FID2, FID3, FID4: Fiducial_1mm_Mask2mm, Fiducial:Fiducial_1mm_Mask2mm
- moved R139 99.5 mm to (120.6, 169.6)
- moved R34 96.8 mm to (122.7, 170.4)
- moved C119 96.4 mm to (112.2, 166.6), turned to 180 degrees
- moved C120 95.6 mm to (112.2, 168.2), turned to 180 degrees
- moved R27 94.0 mm to (120.0, 166.9), turned to 180 degrees
- moved R108 93.8 mm to (118.4, 158.0), turned to 90 degrees
- moved C113 93.3 mm to (115.2, 163.4), turned to 90 degrees
- moved R85 92.6 mm to (122.0, 166.9)
- moved R41 92.4 mm to (113.0, 162.6), turned to -90 degrees
- moved C155 90.7 mm to (129.6, 172.2), turned to 0 degrees
- moved U19 90.2 mm to (116.3, 167.6), turned to 180 degrees
- moved R32 89.4 mm to (117.0, 171.8), turned to 90 degrees
- moved C121 89.2 mm to (116.0, 171.7), turned to -90 degrees
- moved R23 87.6 mm to (114.7, 161.1), turned to 0 degrees
- moved R12 87.6 mm to (120.5, 159.4), turned to -90 degrees
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Routing:
- net /Clock Generator/P2: track 0.00 -> 68.5 mm
- net /Clock Generator/P1: track 0.00 -> 43.4 mm
- net /Clock Generator/CLK2: track 0.00 -> 25.3 mm
- net /Clock Generator/CLK1: track 0.00 -> 17.9 mm, vias 0 -> 3
- net GND: track 0.00 -> 16.8 mm, vias 0 -> 18
- net /Clock Generator/CLK5: track 0.00 -> 15.2 mm, vias 0 -> 2
- net /Clock Generator/CLK6: track 0.00 -> 14.3 mm, vias 0 -> 2
- net /Clock Generator/CLK7: track 0.00 -> 13.6 mm, vias 0 -> 2
- net /Clock Generator/XA: track 0.00 -> 13.6 mm, vias 0 -> 2
- net /Clock Generator/INTR: track 0.00 -> 12.4 mm, vias 0 -> 2
- net /Clock Generator/AUX_CLK2: track 0.00 -> 12.0 mm, vias 0 -> 2
- net /Clock Generator/CLK3: track 0.00 -> 11.6 mm, vias 0 -> 2
- net /Clock Generator/AUX_CLK1: track 0.00 -> 10.6 mm, vias 0 -> 2
- net /Clock Generator/CLK0: track 0.00 -> 10.6 mm, vias 0 -> 2
- net /Clock Generator/CLKIN: track 0.00 -> 10.2 mm
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- added copper zone on F.Cu, net 3V3CLK
- added copper zone on In2.Cu, net 3V3CLK
- added copper zone on In1.Cu, net GND
- added copper zone on In4.Cu, net GND
- added copper zone on F.Cu, net VCC
Other:
- board text removed: "1"
- board text removed: "2"
- board text removed: "3"
- board text removed: "4"
- board text removed: "5"
- board text removed: "6"
- board text removed: "FPGA"
- board text removed: "MCU"
- board text removed: "P3 RF"
