File: fpga/q-radio.kicad_pcb (KiCad board)
At the start: 6 copper layers, 39.9 x 30.5 mm, 34 parts, among them U16 ICE40UP5K

Commit message: All sub-modules added to child projects
Parts:
- moved C117 60.0 mm to (92.5, 115.3), turned to 180 degrees
- moved C178 49.0 mm to (100.1, 110.0)
- moved C183 46.6 mm to (98.0, 116.6), turned to 180 degrees
- moved R21 46.6 mm to (104.4, 107.7), turned to 90 degrees
- moved C174 45.2 mm to (101.9, 110.0), turned to 90 degrees
- moved C185 44.8 mm to (98.0, 117.3), turned to 180 degrees
- moved R145 43.5 mm to (107.1, 109.2), turned to -90 degrees
- moved FB6 42.4 mm to (95.8, 114.8), turned to 180 degrees
- moved RN8 42.1 mm to (102.4, 107.7)
- moved R44 41.6 mm to (105.4, 107.7)
- moved R45 41.4 mm to (109.9, 114.8), turned to 0 degrees
- moved FB8 40.8 mm to (97.8, 108.7)
- moved C177 38.5 mm to (99.3, 110.0), turned to 90 degrees
- moved R40 38.3 mm to (109.9, 113.8)
- moved RN2 38.3 mm to (95.8, 120.9)
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Routing:
- net 1V2FPGA: track 0.00 -> 19.4 mm, vias 0 -> 11
- net 3V3FPGA: track 0.00 -> 13.4 mm, vias 0 -> 14
- net /FPGA/FPGA_DD2: track 0.00 -> 10.3 mm
- net GND: track 0.00 -> 10.1 mm, vias 0 -> 13
- net /FPGA/FPGA_DD5: track 0.00 -> 9.35 mm
- net /FPGA/FPGA_DA2: track 0.00 -> 9.34 mm
- net /FPGA/FPGA_DA1: track 0.00 -> 9.34 mm
- net /FPGA/FPGA_DA0: track 0.00 -> 9.34 mm
- net /FPGA/FPGA_DA3: track 0.00 -> 9.34 mm
- net /FPGA/FPGA_DD0: track 0.00 -> 9.30 mm
- net /FPGA/FPGA_DD1: track 0.00 -> 9.30 mm
- net /FPGA/FPGA_DA6: track 0.00 -> 8.91 mm
- net /FPGA/FPGA_DA7: track 0.00 -> 8.91 mm
- net /FPGA/FPGA_DA5: track 0.00 -> 8.91 mm
- net /FPGA/FPGA_DA4: track 0.00 -> 8.91 mm
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- added copper zone on F.Cu, net /FPGA/VCCPLL
- added copper zone on F.Cu, net 1V2FPGA
- added copper zone on In2.Cu, net 1V2FPGA
- added copper zone on F.Cu, net 2V5FPGA
- added copper zone on F.Cu, net 3V3FPGA
- added copper zone on In2.Cu, net 3V3FPGA
- added copper zone on In1.Cu, net GND
- added copper zone on In4.Cu, net GND
