File: frontend/q-radio.kicad_pcb (KiCad board)
At the start: 6 copper layers, 120 x 75 mm, 73 parts, among them P3 SMA, Q1 NMOS/PMOS, U12 MXD8638C, U13 74LVC1G86, U14 MXD8638C, U24 AP22652, U25 TRF37C73, U40 BGB741L7ESD

Commit message: All sub-modules added to child projects
Parts:
- removed FID1, FID2, FID3, FID4: Fiducial_1mm_Mask2mm, Fiducial:Fiducial_1mm_Mask2mm
Routing:
- net GND: track 0.00 -> 26.9 mm, vias 0 -> 35
- net /RF Front End/~{RX_AMP_EN}: track 0.00 -> 19.7 mm, vias 0 -> 3
- net /RF Front End/~{TX_AMP_EN}: track 0.00 -> 16.5 mm, vias 0 -> 3
- net /RF Front End/AMP_BYPASS: track 0.00 -> 10.8 mm
- net VAA: track 0.00 -> 10.2 mm, vias 0 -> 16
- net Net-(D1-A1): track 0.00 -> 8.57 mm
- net Net-(D15-K): track 0.00 -> 6.32 mm
- net Net-(U40-BIAS): track 0.00 -> 5.62 mm, vias 0 -> 2
- net Net-(U40-RFIN): track 0.00 -> 4.76 mm
- net Net-(C207-Pad1): track 0.00 -> 4.67 mm
- net /RF Front End/BIAS: track 0.00 -> 4.51 mm
- net Net-(U40-RFOUT): track 0.00 -> 4.47 mm
- net Net-(C210-Pad1): track 0.00 -> 4.42 mm
- net Net-(C139-Pad1): track 0.00 -> 3.88 mm
- net /RF Front End/RX_AMP_EN: track 0.00 -> 3.86 mm, vias 0 -> 2
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- added copper zone on B.Cu, net 2V5RF
- added copper zone on F.Cu, net 2V5RF
- added copper zone on In1.Cu, net GND
- added copper zone on In4.Cu, net GND
- added copper zone on F.Cu, net VAA
- added copper zone on In2.Cu, net VAA
Other:
- board size 120 x 75 mm -> 27.5 x 21.3 mm
- board text removed: "1"
- board text removed: "3"
- board text removed: "4"
- board text removed: "6"
