File: if-transceiver/q-radio.kicad_pcb (KiCad board)
At the start: 6 copper layers, 120 x 75 mm, 43 parts, among them T3 IF_BALUN, T4 IF_BALUN, U17 MAX2831, U2 MXD8546F, U7 FM8625H

Commit message: All sub-modules added to child projects
Parts:
- removed FID1, FID2, FID3, FID4: Fiducial_1mm_Mask2mm, Fiducial:Fiducial_1mm_Mask2mm
Routing:
- net GND: track 0.00 -> 49.3 mm, vias 0 -> 31
- net VAA: track 0.00 -> 19.1 mm, vias 0 -> 17
- net /IF Transceiver/TUNE: track 0.00 -> 7.20 mm, vias 0 -> 2
- net /IF Transceiver/IF: track 0.00 -> 6.78 mm
- net /IF Transceiver/XTAL: track 0.00 -> 3.95 mm
- net /IF Transceiver/CPOUT: track 0.00 -> 3.00 mm
- net /IF Transceiver/RXIF: track 0.00 -> 2.66 mm
- net Net-(FL3-IN): track 0.00 -> 2.04 mm
- net /IF Transceiver/XCVR.~{SHDN}: track 0.00 -> 1.87 mm
- net Net-(FL2-IN): track 0.00 -> 1.85 mm
- net /IF Transceiver/TXIF_BALUN+: track 0.00 -> 1.58 mm
- net /IF Transceiver/RXIF_BALUN+: track 0.00 -> 1.58 mm
- net 2V5RF: track 0.00 -> 1.55 mm, vias 0 -> 4
- net /IF Transceiver/TXIF_BALUN-: track 0.00 -> 1.55 mm
- net /IF Transceiver/RXIF_BALUN-: track 0.00 -> 1.55 mm
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- added copper zone on In2.Cu, net 2V5RF
- added copper zone on In1.Cu, net GND
- added copper zone on In4.Cu, net GND
- added copper zone on B.Cu, net VAA
- added copper zone on F.Cu, net VAA
- added copper zone on In2.Cu, net VAA
Other:
- board size 120 x 75 mm -> 29.5 x 19.4 mm
- board text removed: "1"
- board text removed: "2"
- board text removed: "3"
- board text removed: "4"
- board text removed: "5"
- board text removed: "6"
- board text removed: "P3 RF"
