File: mcu/q-radio.kicad_pcb (KiCad board)
At the start: 6 copper layers, 60.1 x 68.3 mm, 49 parts, among them P20 HEADER_2x11, P22 HEADER_2x13, P26 LPC_JTAG, P28 HEADER_2x11, U20 W25Q32, U23 LPC4330FET180, X2 MCU_XTAL, X3 RTC_XTAL

Commit message: All sub-modules added to child projects
Parts:
- removed FID1, FID2, FID3, FID4: Fiducial_1mm_Mask2mm, Fiducial:Fiducial_1mm_Mask2mm
- moved R62 80.3 mm to (143.6, 101.6), turned to 0 degrees
- moved C138 71.7 mm to (146.9, 150.7), turned to -90 degrees
- moved R127 71.6 mm to (127.7, 139.4), turned to 0 degrees
- moved R107 67.9 mm to (155.1, 133.9), turned to 0 degrees
- moved C131 67.6 mm to (139.3, 144.3), turned to 180 degrees
- moved R6 65.4 mm to (128.1, 138.1)
- moved R141 65.0 mm to (136.9, 142.4)
- moved R68 64.4 mm to (137.5, 152.3), turned to 180 degrees
- moved R65 64.3 mm to (139.6, 101.6)
- moved C130 64.0 mm to (148.7, 150.8), turned to -90 degrees
- moved C158 63.7 mm to (150.3, 128.1), turned to 90 degrees
- moved R93 61.7 mm to (139.1, 154.2), turned to 0 degrees
- moved C134 61.2 mm to (150.6, 150.8), turned to -90 degrees
- moved C157 61.0 mm to (152.5, 128.1)
- moved C128 60.5 mm to (147.9, 132.6), turned to 90 degrees
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Routing:
- net /Microcontroller/~{RESET}: track 0.00 -> 132.8 mm, vias 0 -> 1
- net /Microcontroller/P5_7: track 0.00 -> 43.3 mm
- net /Microcontroller/USB0_VBUS: track 0.00 -> 41.1 mm
- net /Microcontroller/TDI: track 0.00 -> 39.8 mm, vias 0 -> 1
- net /Microcontroller/I2C1_SCL: track 0.00 -> 38.9 mm, vias 0 -> 1
- net /Microcontroller/I2C1_SDA: track 0.00 -> 38.5 mm, vias 0 -> 1
- net /Microcontroller/TCK: track 0.00 -> 37.8 mm, vias 0 -> 2
- net /Microcontroller/TMS: track 0.00 -> 37.6 mm, vias 0 -> 1
- net /Microcontroller/TDO: track 0.00 -> 36.8 mm, vias 0 -> 2
- net /Microcontroller/PA_4: track 0.00 -> 36.4 mm, vias 0 -> 1
- net GND: track 0.00 -> 33.8 mm, vias 0 -> 36
- net /Microcontroller/SD_DAT2: track 0.00 -> 33.7 mm
- net /Microcontroller/DBGEN: track 0.00 -> 33.7 mm, vias 0 -> 2
- net /Microcontroller/P2_9: track 0.00 -> 33.5 mm, vias 0 -> 2
- net /Microcontroller/GPIO3_15: track 0.00 -> 32.3 mm, vias 0 -> 1
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- added copper zone on In2.Cu, net 3V3AUX
- added copper zone on In1.Cu, net GND
- added copper zone on In4.Cu, net GND
- added copper zone on F.Cu, net VCC
- added copper zone on In2.Cu, net VCC
