File: mcu/mcu.kicad_sch (KiCad schematic)
At the start: 45 parts, among them P20 HEADER_2x11, P22 HEADER_2x13, P26 LPC_JTAG, P28 HEADER_2x11, U20 W25Q32, U23 LPC4330FET180, X2 MCU_XTAL, X3 RTC_XTAL

Commit message: separated LED and SW subcircuit as it's pre-placed and not part of MCU room. Updated all other sch subcircuits.
Changed lines of the file:
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@@
 	)
 	(bus_entry
+		(at 44.45 129.54)
+		(size 2.54 2.54)
+		(stroke
+			(width 0)
+			(type default)
+		)
+	)
+	(bus_entry
 		(at 384.81 223.52)
 		(size 2.54 2.54)
@@
 	)
 	(bus_entry
+		(at 44.45 133.35)
+		(size 2.54 2.54)
+		(stroke
+			(width 0)
+			(type default)
+		)
+	)
+	(bus_entry
 		(at 157.48 182.88)
 		(size -2.54 -2.54)
@@
 	)
 	(bus_entry
+		(at 44.45 140.97)
+		(size 2.54 2.54)
+		(stroke
+			(width 0)
+			(type default)
+		)
+	)
+	(bus_entry
 		(at 383.54 59.69)
 		(size 2.54 2.54)
@@
 	)
 	(bus_entry
+		(at 44.45 137.16)
+		(size 2.54 2.54)
+		(stroke
+			(width 0)
+			(type default)
+		)
+	)
+	(bus_entry
 		(at 383.54 46.99)
 		(size 2.54 2.54)
@@
 		)
 	)
+	(bus
+		(pts
+			(xy 44.45 129.54) (xy 44.45 133.35)
+		)
+		(stroke
+			(width 0)
+			(type default)
+		)
+	)
 	(wire
 		(pts
@@
 		)
 	)
+	(bus
+		(pts
+			(xy 36.83 129.54) (xy 44.45 129.54)
+		)
+		(stroke
+			(width 0)
+			(type default)
+		)
+	)
 	(wire
 		(pts
@@
 	(wire
 		(pts
-			(xy 194.31 114.3) (xy 187.96 114.3)
-		)
-		(stroke
-			(width 0)
-			(type default)
-		)
-	)
-	(wire
-		(pts
 			(xy 130.81 105.41) (xy 133.35 105.41)
 		)
@@
 	(wire
 		(pts
+			(xy 168.91 114.3) (xy 194.31 114.3)
+		)
+		(stroke
+			(width 0)
+			(type default)
+		)
+	)
+	(wire
+		(pts
 			(xy 245.11 73.66) (xy 252.73 73.66)
 		)
@@
 	(wire
 		(pts
+			(xy 46.99 139.7) (xy 57.15 139.7)
+		)
+		(stroke
+			(width 0)
+			(type default)
+		)
+	)
+	(wire
+		(pts
 			(xy 245.11 134.62) (xy 264.16 134.62)
 		)
@@
 	(wire
 		(pts
+			(xy 46.99 143.51) (xy 57.15 143.51)
+		)
+		(stroke
+			(width 0)
+			(type default)
+		)
+	)
+	(wire
+		(pts
 			(xy 194.31 43.18) (xy 186.69 43.18)
 		)
@@
 	(bus
 		(pts
+			(xy 44.45 133.35) (xy 44.45 140.97)
+		)
+		(stroke
+			(width 0)
+			(type default)
+		)
+	)
+	(bus
+		(pts
 			(xy 386.08 54.61) (xy 386.08 57.15)
 		)
@@
 	(wire
 		(pts
+			(xy 46.99 135.89) (xy 57.15 135.89)
+		)
+		(stroke
+			(width 0)
+			(type default)
+		)
+	)
+	(wire
+		(pts
 			(xy 365.76 147.32) (xy 377.19 147.32)
 		)
@@
 	(wire
 		(pts
+			(xy 46.99 132.08) (xy 57.15 132.08)
+		)
+		(stroke
+			(width 0)
+			(type default)
+		)
+	)
+	(wire
+		(pts
 			(xy 377.19 137.16) (xy 365.76 137.16)
 		)
@@
 		)
 	)
+	(label "~{LED2}"
+		(at 49.53 135.89 0)
+		(effects
+			(font
+				(size 1.27 1.27)
+			)
+			(justify left bottom)
+		)
+	)
 	(label "ADC0_3"
 		(at 252.73 218.44 180)
@@
 		)
 	)
+	(label "~{LED5}"
+		(at 49.53 143.51 0)
+		(effects
+			(font
+				(size 1.27 1.27)
+			)
+			(justify left bottom)
+		)
+	)
 	(label "GPIO3_12"
 		(at 369.57 111.76 0)
@@
 		)
 	)
+	(label "~{LED1}"
+		(at 49.53 132.08 0)
+		(effects
+			(font
+				(size 1.27 1.27)
+			)
+			(justify left bottom)
+		)
+	)
 	(label "P2_9"
 		(at 187.96 116.84 0)
@@
 		)
 	)
+	(label "~{LED3}"
+		(at 49.53 139.7 0)
+		(effects
+			(font
+				(size 1.27 1.27)
+			)
+			(justify left bottom)
+		)
+	)
 	(label "GPIO3_14"
 		(at 186.69 248.92 0)
@@
 		)
 	)
+	(hierarchical_label "~{LED[1..4]}"
+		(shape output)
+		(at 36.83 129.54 180)
+		(effects
+			(font
+				(size 1.27 1.27)
+			)
+			(justify right)
+		)
+	)
 	(hierarchical_label "VIN"
 		(shape output)
@@
 		)
 	)
+	(hierarchical_label "~{RESET}"
+		(shape passive)
+		(at 254 198.12 0)
+		(effects
+			(font
+				(size 1.27 1.27)
+			)
+			(justify left)
+		)
+	)
 	(hierarchical_label "XCVR{MAX2831}"
 		(shape bidirectional)
@@
 		)
 	)
+	(hierarchical_label "P2_8"
+		(shape passive)
+		(at 168.91 114.3 180)
+		(effects
+			(font
+				(size 1.27 1.27)
+			)
+			(justify right)
+		)
+	)
 	(hierarchical_label "SCT_CLK"
 		(shape input)
@@
 		(polyline
 			(pts
-				(xy 77.47 199.39) (xy 157.48 199.39) (xy 157.48 220.98) (xy 124.46 220.98) (xy 124.46 243.84) (xy 105.41 243.84)
-				(xy 105.41 264.16) (xy 77.47 264.16)
-			)
-			(stroke
-				(width 0)
-				(type dash)
-			)
-			(fill
-				(type none)
-			)
-		)
-	)
-	(rule_area
-		(exclude_from_sim no)
-		(in_bom yes)
-		(on_board yes)
-		(dnp no)
-		(polyline
-			(pts
-				(xy 337.82 118.11) (xy 292.1 118.11) (xy 292.1 132.08) (xy 270.51 132.08) (xy 265.43 137.16) (xy 265.43 189.23)
-				(xy 336.55 189.23) (xy 337.82 162.56)
+				(xy 19.05 15.24) (xy 19.05 48.26) (xy 120.65 48.26) (xy 120.65 231.14) (xy 134.62 231.14) (xy 134.62 264.16)
+				(xy 297.18 264.16) (xy 297.18 104.14) (xy 281.94 104.14) (xy 281.94 15.24)
 			)
 			(stroke
@@
 		(length 2.54)
 		(shape round)
-		(at 83.82 199.39 0)
-		(fields_autoplaced yes)
-		(effects
-			(font
-				(size 1.27 1.27)
-			)
-			(justify left bottom)
-		)
-		(property "Netclass" ""
-			(at 204.47 30.48 0)
-			(show_name no)
-			(do_not_autoplace no)
-			(effects
-				(font
-					(size 1.27 1.27)
-				)
-			)
-		)
-		(property "Component Class" "JUMPERS"
-			(at 84.5185 196.85 0)
-			(show_name no)
-			(do_not_autoplace no)
-			(effects
-				(font
-					(size 1.27 1.27)
-					(italic yes)
-				)
-				(justify left)
-			)
-		)
-	)
-	(netclass_flag ""
-		(length 2.54)
-		(shape round)
-		(at 328.93 118.11 0)
+		(at 281.94 99.06 270)
 		(fields_autoplaced yes)
 		(effects
 			(font
-				(size 1.27 1.27)
+				(size 1.524 1.524)
 			)
-			(justify left bottom)
+			(justify right bottom)
 		)
 		(property "Netclass" ""
-			(at 105.41 8.89 0)
+			(at 377.19 45.72 0)
 			(show_name no)
 			(do_not_autoplace no)
@@
 			)
 		)
-		(property "Component Class" "JTAG"
-			(at 329.6285 115.57 0)
+		(property "Component Class" "Microcontroller"
+			(at 284.48 98.4301 90)
 			(show_name no)
 			(do_not_autoplace no)
