File: mixer/q-radio.kicad_pcb (KiCad board)
At the start: 6 copper layers, 120 x 75 mm, 80 parts, among them T1 RF_BALUN, T2 RF_BALUN, U38 BGB741L7ESD, U4 RFFC5072, U5 FM8625H, U6 FM8625H

Commit message: All sub-modules added to child projects
Parts:
- removed FID1, FID2, FID4: Fiducial_1mm_Mask2mm, Fiducial:Fiducial_1mm_Mask2mm
Routing:
- net Net-(U5-RF1): track 0.00 -> 26.2 mm
- net GND: track 0.00 -> 21.7 mm, vias 0 -> 30
- net /Mixer/RX_EN: track 0.00 -> 11.3 mm, vias 0 -> 2
- net VAA: track 0.00 -> 10.2 mm, vias 0 -> 12
- net Net-(C188-Pad1): track 0.00 -> 8.46 mm
- net /Mixer/MIXER.~{RESET}: track 0.00 -> 6.52 mm, vias 0 -> 2
- net /Mixer/MIX_OUT-: track 0.00 -> 5.19 mm
- net /Mixer/MIX_OUT+: track 0.00 -> 5.19 mm
- net Net-(C195-Pad1): track 0.00 -> 4.35 mm
- net /Mixer/MIXER.~{EN}: track 0.00 -> 4.35 mm
- net Net-(C191-Pad1): track 0.00 -> 4.31 mm
- net Net-(U38-BIAS): track 0.00 -> 3.75 mm
- net Net-(C202-Pad2): track 0.00 -> 3.74 mm
- net Net-(C203-Pad1): track 0.00 -> 3.66 mm
- net /Mixer/MIXER.SCLK: track 0.00 -> 3.45 mm
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- added copper zone on In2.Cu, net 2V5RF
- added copper zone on In1.Cu, net GND
- added copper zone on In4.Cu, net GND
- added copper zone on F.Cu, net VAA
- added copper zone on In2.Cu, net VAA
Other:
- board size 120 x 75 mm -> 26.3 x 19.1 mm
- board text removed: "1"
- board text removed: "2"
- board text removed: "3"
- board text removed: "4"
- board text removed: "5"
- board text removed: "6"
