File: power/q-radio.kicad_pcb (KiCad board)
At the start: 6 copper layers, 82 x 33 mm, 85 parts, among them Q10 2NPN, Q3 PMOS, Q4 PMOS, Q5 PMOS, Q6 PMOS, Q7 2NPN, Q9 2PNP, U21 TPS62410, U22 LDO_2V5, U28 AP22652, U32 LDO_2V5

Commit message: All sub-modules added to child projects
Parts:
- removed FID4: Fiducial_1mm_Mask2mm, Fiducial:Fiducial_1mm_Mask2mm
- moved C175 107.8 mm to (114.4, 106.1), turned to 180 degrees
- moved FB7 104.6 mm to (124.2, 105.4)
- moved C172 103.4 mm to (124.9, 108.6), turned to -90 degrees
- moved R53 103.3 mm to (118.3, 113.0), turned to -90 degrees
- moved C184 101.9 mm to (122.4, 108.6), turned to -90 degrees
- moved U22 100.9 mm to (118.6, 107.3), turned to -90 degrees
- moved Q7 99.7 mm to (118.3, 115.7), turned to -90 degrees
- moved Q6 98.9 mm to (122.0, 116.5), turned to 180 degrees
- moved C165 96.6 mm to (129.1, 108.0), turned to 90 degrees
- moved R61 96.5 mm to (124.9, 116.5), turned to -90 degrees
- moved R71 95.3 mm to (119.1, 118.3)
- moved C181 95.3 mm to (117.7, 110.7)
- moved FB4 95.1 mm to (120.7, 112.9)
- moved C173 95.1 mm to (119.4, 113.0), turned to -90 degrees
- moved C166 93.2 mm to (124.4, 122.6), turned to 180 degrees
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Routing:
- net GND: track 0.00 -> 38.3 mm, vias 0 -> 41
- net Net-(D13-A): track 0.00 -> 16.4 mm
- net Net-(Q10A-C1): track 0.00 -> 13.3 mm
- net +1V2: track 0.00 -> 11.3 mm, vias 0 -> 4
- net Net-(U21-DEF_1): track 0.00 -> 10.0 mm
- net +5V: track 0.00 -> 9.47 mm
- net /Power/MODE: track 0.00 -> 9.46 mm
- net Net-(U21-EN1): track 0.00 -> 9.32 mm, vias 0 -> 2
- net /Power/VRM_IN: track 0.00 -> 9.17 mm
- net Net-(D17-K): track 0.00 -> 9.01 mm
- net VCC: track 0.00 -> 8.59 mm, vias 0 -> 17
- net /Power/~{3V3AUX_EN}: track 0.00 -> 7.34 mm
- net Net-(Q6-G): track 0.00 -> 7.25 mm
- net Net-(Q3-D): track 0.00 -> 5.82 mm
- net Net-(U21-ADJ2): track 0.00 -> 4.48 mm
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- added copper zone on F.Cu, net +1V2
- added copper zone on F.Cu, net +2V5
- added copper zone on F.Cu, net /Power/VBUS
- added copper zone on B.Cu, net /Power/VBUS_SAFE
- added copper zone on F.Cu, net /Power/VBUS_SAFE
- added copper zone on F.Cu, net /Power/VIN
- added copper zone on F.Cu, net /Power/VRM_IN
- added copper zone on F.Cu, net /Power/VSW_1
- added copper zone on F.Cu, net /Power/VSW_2
- added copper zone on F.Cu, net 1V2FPGA
- added copper zone on F.Cu, net 2V5RF
- added copper zone on F.Cu, net 3V3AUX
- added copper zone on F.Cu, net 3V3CLK
- added copper zone on B.Cu, net 3V3FPGA
- added copper zone on F.Cu, net 3V3FPGA
- added copper zone on F.Cu, net 3V3LED
- added copper zone on In1.Cu, net GND
- added copper zone on In4.Cu, net GND
- added copper zone on F.Cu, net Net-(D13-A)
- added copper zone on F.Cu, net Net-(Q6-D)
- added copper zone on F.Cu, net VAA
- added copper zone on F.Cu, net VCC
- added copper zone on In2.Cu, net VCC
Other:
- board text removed: "1"
- board text removed: "2"
- board text removed: "3"
- board text removed: "4"
- board text removed: "5"
- board text removed: "6"
