File: usb/q-radio.kicad_pcb (KiCad board)
At the start: 6 copper layers, 18 x 14.7 mm, 10 parts, among them J1 USB_C, U15 TVS_USB

Commit message: All sub-modules added to child projects
Parts:
- moved D18 65.3 mm to (105.7, 128.2), turned to 0 degrees
- moved C152 63.8 mm to (106.4, 119.1), turned to 180 degrees
- moved U15 61.1 mm to (109.5, 122.0), turned to 0 degrees
- moved R157 60.8 mm to (104.2, 121.4)
- moved R156 59.9 mm to (105.9, 116.3), turned to 180 degrees
- moved R106 58.7 mm to (106.4, 118.2), turned to 0 degrees
- moved C151 58.7 mm to (108.3, 118.3), turned to 90 degrees
- moved R103 56.2 mm to (109.3, 118.3), turned to -90 degrees
- moved FL1 4.12 mm to (107.0, 122.7)
Connections:
- FL1 pad 1: /USB/USB_DATA.D- -> /USB/USB_DATA.D+
- FL1 pad 2: /USB/D- -> /USB/D+
- FL1 pad 3: /USB/USB_DATA.D+ -> /USB/USB_DATA.D-
- FL1 pad 4: /USB/D+ -> /USB/D-
- U15 pad 1: /USB/CC1 -> /USB/CC2
- U15 pad 10: /USB/CC1 -> /USB/CC2
- U15 pad 2: /USB/CC2 -> /USB/CC1
- U15 pad 9: /USB/CC2 -> /USB/CC1
Routing:
- net /USB/CC1: track 0.00 -> 11.1 mm, vias 0 -> 2
- net /USB/D+: track 0.00 -> 8.02 mm
- net /USB/D-: track 0.00 -> 8.02 mm
- net /USB/VBUS: track 0.00 -> 7.94 mm, vias 0 -> 5
- net GND: track 0.00 -> 7.58 mm, vias 0 -> 6
- net /USB/CC2: track 0.00 -> 7.01 mm
- net /USB/ADC0_4: track 0.00 -> 4.10 mm
- net /USB/ADC0_7: track 0.00 -> 4.07 mm
- added copper zone on F.Cu, net /USB/VBUS
- added copper zone on In2.Cu, net /USB/VBUS
- added copper zone on In1.Cu, net GND
- added copper zone on In4.Cu, net GND
